File: Adlib.sch (KiCad schematic (older format))
At the start: 60 parts, among them J1 CONN_01X05, P1 IRQ, P2 ADDR, Q1 2N3904, U1 74LS109, U2 74LS138, U3 74LS138, U4 74LS245, U5 74LS04, U6 YM3812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

Commit message: Update title block, add libs, add pdf
Parts:
- R14: symbol POT -> POT-RESCUE-Adlib
Changed lines of the file:
@@
 EESchema Schematic File Version 2
+LIBS:Adlib-rescue
 LIBS:power
 LIBS:device
@@
 encoding utf-8
 Sheet 1 1
-Title ""
+Title "Reproduction AdLib Sound Card, OPL2, Circa 1990"
 Date ""
 Rev ""
 Comp ""
-Comment1 ""
-Comment2 ""
-Comment3 ""
+Comment1 "Copyright (C) 2017 Eric Schlaepfer"
+Comment2 "See https://creativecommons.org/licenses/by/4.0/"
+Comment3 "This work is licensed under a Creative Commons Attribution 4.0 International License. "
 Comment4 ""
 $EndDescr
@@
 $EndComp
 $Comp
-L POT R14
+L POT-RESCUE-Adlib R14
 U 1 1 57774901
 P 8100 5850
